File: prueba/PULSAR/PULSAR.kicad_sch (KiCad schematic)
At the start: 12 parts, among them J1 Conn_01x20, J2 Conn_01x20, J3 USB_C_Receptacle, J4 Conn_01x07, U1 AP2112K-3.3, U2 SS49E, U3 CD74HC4067M, U4 ADS8688

Commit message: feat: PCB routing in progress - power and SPI connections
Parts:
- C1, C2: LCSC (none) -> C52923
- J1, J2: footprint (none) -> Connector_PinHeader_2.54mm:PinHeader_1x20_P2.54mm_Vertical; now left out of the parts list
- J3: LCSC (none) -> C168688
- J4: footprint (none) -> Connector_PinHeader_2.54mm:PinHeader_1x07_P2.54mm_Vertical; now left out of the parts list
- R_CC1, R_CC2: footprint (none) -> Resistor_SMD:R_0402_1005Metric; LCSC (none) -> C23186
- U1: LCSC (none) -> C51118
- U2: LCSC (none) -> C85697
- U3: footprint Package_SO:SOIC-24W_7.5x15.4mm_P1.27mm -> Package_SO:SSOP-24_5.3x8.2mm_P0.65mm; LCSC (none) -> C98457
- U4: LCSC (none) -> C1542682
Connections:
- net SPI__CS0 is gone; now on net SPI_CS0: J1.6 (Pin_6)
- net SPI__MISO is gone; now on net SPI_SDO: J1.5 (Pin_5)
Changed lines of the file:
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@@
 		)
 	)
-	(label "SPI__CS0"
+	(label "SPI_CS0"
 		(at 78.74 43.18 0)
 		(effects
@@
 		)
 	)
-	(label "SPI__MISO"
+	(label "SPI_SDO"
 		(at 78.74 40.64 0)
 		(effects
@@
 			)
 		)
-		(property "Footprint" ""
+		(property "Footprint" "Resistor_SMD:R_0402_1005Metric"
 			(at 59.69 50.038 90)
 			(hide yes)
@@
 			)
 		)
+		(property "LCSC" "C23186"
+			(at 59.69 48.26 90)
+			(hide yes)
+			(show_name no)
+			(do_not_autoplace no)
+			(effects
+				(font
+					(size 1.27 1.27)
+				)
+			)
+		)
 		(pin "2"
 		)
@@
 			)
 		)
+		(property "LCSC" "C85697"
+			(at 171.45 152.4 0)
+			(hide yes)
+			(show_name no)
+			(do_not_autoplace no)
+			(effects
+				(font
+					(size 1.27 1.27)
+				)
+			)
+		)
 		(pin "3"
 		)
@@
 			)
 		)
-		(property "Footprint" ""
+		(property "Footprint" "Resistor_SMD:R_0402_1005Metric"
 			(at 53.34 52.578 90)
 			(hide yes)
@@
 			)
 		)
+		(property "LCSC" "C23186"
+			(at 53.34 50.8 90)
+			(hide yes)
+			(show_name no)
+			(do_not_autoplace no)
+			(effects
+				(font
+					(size 1.27 1.27)
+				)
+			)
+		)
 		(pin "2"
 		)
@@
 		(body_style 1)
 		(exclude_from_sim no)
-		(in_bom yes)
+		(in_bom no)
 		(on_board yes)
 		(in_pos_files yes)
@@
 			)
 		)
-		(property "Footprint" ""
+		(property "Footprint" "Connector_PinHeader_2.54mm:PinHeader_1x20_P2.54mm_Vertical"
 			(at 130.81 53.34 0)
 			(hide yes)
@@
 			)
 		)
+		(property "LCSC" "C51118"
+			(at 209.55 137.16 0)
+			(hide yes)
+			(show_name no)
+			(do_not_autoplace no)
+			(effects
+				(font
+					(size 1.27 1.27)
+				)
+			)
+		)
 		(pin "4"
 		)
@@
 			)
 		)
+		(property "LCSC" "C52923"
+			(at 223.52 149.86 0)
+			(hide yes)
+			(show_name no)
+			(do_not_autoplace no)
+			(effects
+				(font
+					(size 1.27 1.27)
+				)
+			)
+		)
 		(pin "1"
 		)
@@
 			)
 		)
+		(property "LCSC" "C52923"
+			(at 194.31 149.86 0)
+			(hide yes)
+			(show_name no)
+			(do_not_autoplace no)
+			(effects
+				(font
+					(size 1.27 1.27)
+				)
+			)
+		)
 		(pin "1"
 		)
@@
 			)
 		)
+		(property "LCSC" "C168688"
+			(at 27.94 68.58 0)
+			(hide yes)
+			(show_name no)
+			(do_not_autoplace no)
+			(effects
+				(font
+					(size 1.27 1.27)
+				)
+			)
+		)
 		(pin "A4"
 		)
@@
 			)
 		)
-		(property "Footprint" "Package_SO:SOIC-24W_7.5x15.4mm_P1.27mm"
+		(property "Footprint" "Package_SO:SSOP-24_5.3x8.2mm_P0.65mm"
 			(at 156.21 182.88 0)
 			(hide yes)
@@
 			)
 		)
+		(property "LCSC" "C98457"
+			(at 133.35 157.48 0)
+			(hide yes)
+			(show_name no)
+			(do_not_autoplace no)
+			(effects
+				(font
+					(size 1.27 1.27)
+				)
+			)
+		)
 		(pin "11"
 		)
@@
 		(body_style 1)
 		(exclude_from_sim no)
-		(in_bom yes)
+		(in_bom no)
 		(on_board yes)
 		(in_pos_files yes)
@@
 			)
 		)
-		(property "Footprint" ""
+		(property "Footprint" "Connector_PinHeader_2.54mm:PinHeader_1x07_P2.54mm_Vertical"
 			(at 264.16 130.81 0)
 			(hide yes)
@@
 		(body_style 1)
 		(exclude_from_sim no)
-		(in_bom yes)
+		(in_bom no)
 		(on_board yes)
 		(in_pos_files yes)
@@
 			)
 		)
-		(property "Footprint" ""
+		(property "Footprint" "Connector_PinHeader_2.54mm:PinHeader_1x20_P2.54mm_Vertical"
 			(at 93.98 53.34 0)
 			(hide yes)
@@
 			(at 209.55 74.93 0)
 			(hide yes)
+			(show_name no)
+			(do_not_autoplace no)
+			(effects
+				(font
+					(size 1.27 1.27)
+				)
+			)
+		)
+		(property "LCSC" "C1542682"
+			(at 209.55 74.93 0)
+			(hide yes)
