File: pcb/pulsar /adc.kicad_sch (KiCad schematic)
At the start: 0 parts

Commit message: feat: added the pcb of the pulsar
Parts:
- added C1, C3: 1uF 10V X5R 0402, symbol Device:C
- added C10, C11, C12, C13, C2, C20, C22, C24, C26, C28, C30, C32, C34, C4: 100nF 10V X5R 0402, symbol Device:C
- added C21, C23, C25, C27, C29, C31, C33, C35: 10uF 10V X5R 0603, symbol Device:C
- added U1, U2: REF5025AIDR, symbol PULSAR:REF5025
- added U10, U7, U8, U9: ADG1606BRUZ-REEL7, symbol PULSAR:ADG1606
- added U11, U12, U13, U14, U15, U16, U17, U18: AD7689BCPZRL7, symbol PULSAR:AD7689
- added U3, U4, U5, U6: OPA2365AIDR, symbol PULSAR:OPA2365
Connections:
- new net +3.3V: U1.1 (IN), U10.20 (A2), U2.1 (IN), U3.8 (VDD), U4.8 (VDD), U5.8 (VDD), U6.8 (VDD), U7.20 (A2), U8.20 (A2), U9.20 (A2)
- new net GND: U1.2 (GND), U10.15 (VSS), U11.10 (GND), U11.9 (COM), U12.10 (GND), U12.9 (COM), U13.10 (GND), U13.9 (COM), U14.10 (GND), U14.9 (COM), U15.10 (GND), U15.9 (COM), U16.10 (GND), U16.9 (COM), U17.10 (GND), U17.9 (COM), U18.10 (GND), U18.9 (COM), U2.2 (GND), U3.5 (IN+B), U4.5 (IN+B), U5.5 (IN+B), U6.5 (IN+B), U7.15 (VSS), U8.15 (VSS), U9.15 (VSS)
- no-connect marks 0 -> 26
Other:
- note added: "16-bit SAR ADC — AD7689BCPZRL7 (C706705)"
- note added: "16:1 Analog Mux — ADG1606BRUZ-REEL7 (C208204)"
- note added: "Op-Amp Buffers — OPA2365AIDR (C130011)"
- note added: "Voltage References — REF5025AIDR 2.5V (C11341)"
