File: pcb/pulsar /fido2.kicad_sch (KiCad schematic)
At the start: 0 parts

Commit message: feat: added the pcb of the pulsar
Parts:
- added C1, C2, C4, C6: 100nF 10V X5R, symbol Device:C
- added C3: 100nF, symbol Device:C
- added C5: 10uF 10V X5R 0603, symbol Device:C
- added J1: FPC_10P_0.5mm, symbol PULSAR:FPC_10P
- added R1, R2, R3, R4, R5, R6: 4.7k 0402, symbol Device:R
- added U1: ISO1540DR, symbol PULSAR:ISO1540
- added U2: STM32L052K8T6, symbol PULSAR:STM32L052K8T6
- added U3: ATECC608B-MAHDA-S, symbol PULSAR:ATECC608B
Connections:
- new net: C3.1, U2.4 (NRST)
- new net +1V8: R3.1, R3.2, R4.1, R5.1, R5.2, R6.1, U1.5 (VCC2), U2.1 (VDD), U2.32 (VDD), U3.5 (SDA)
- new net +3.3V: J1.2, R1.1, R1.2, R2.1
- new net FIDO2_SCL: R2.2
- new net GND: J1.1, U1.4 (VCC1), U1.6 (GND2), U2.15 (PB1), U2.16 (VSS), U2.31 (BOOT0), U3.1 (NC)
- new net ISO_SDA: R4.2
- new net SEC_SCL: R6.2
- no-connect marks 0 -> 10
Other:
- note added: "FIDO2 Sub-Board (25×30mm) — FPC 10p 0.5mm interface (C460012)"
- note added: "FPC 10p 0.5mm"
