File: pcb/pulsar /fpga_b2.kicad_sch (KiCad schematic)
At the start: 0 parts

Commit message: feat: added the pcb of the pulsar
Parts:
- added C1, C10, C11, C12, C13, C14, C15, C16, C17, C18, C19, C2, C20, C21, C22, C23, C24, C25, C26, C27, C28, C29, C3, C30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: 100nF 10V X5R 0402, symbol Device:C
Other:
- note added: "+1V0 VCCINT (40× 100nF)"
- note added: "+1V0_MGT VCCMGTAVCC (10× 100nF)"
- note added: "+1V2_MGT VCCMGTAVTT (8× 100nF)"
- note added: "+1V8 VCCAUX (10× 100nF)"
- note added: "+2V5_MGT MGTVCCAUX (7× 100nF)"
- note added: "+3.3V VCCO (10× 100nF)"
