File: pcb/pulsar /fpga_c3.kicad_sch (KiCad schematic)
At the start: 0 parts

Commit message: feat: added the pcb of the pulsar
Parts:
- added C1, C6: 100nF 10V X5R 0402, symbol Device:C
- added C2, C3, C4, C5: 18pF 0402, symbol Device:C
- added R1, R2: 10k 0402, symbol Device:R
- added U8: W25Q128JVSIQ, symbol PULSAR:W25Q128JVSIQ
- added U9: IS61WV102416BLL, symbol PULSAR:IS61WV102416BLL
- added Y1: 50MHz, symbol PULSAR:Crystal
- added Y2: 48MHz, symbol PULSAR:Crystal
Connections:
- new net +3.3V: R1.1, R2.1, U8.8 (VCC), U9.44 (VCC)
- new net GND: U8.4 (GND), U9.22 (GND)
