File: pcb/pulsar /hall.kicad_sch (KiCad schematic)
At the start: 0 parts

Commit message: feat: added the pcb of the pulsar
Parts:
- added C1, C10, C100, C101, C102, C103, C104, C105, C106, C107, C108, C109, C11, C110, C111, C112, C113, C114, C115, C116, C117, C118, C119, C12, C120, C121, C122, C13, C14, C15, C16, C17, C18, C19, C2, C20, C21, C22, C23, C24, C25, C26, C27, C28, C29, C3, C30, C31, C32, C33, C34, C35, C36, C37, C38, C39, C4, C40, C41, C42, C43, C44, C45, C46, C47, C48, C49, C5, C50, C51, C52, C53, C54, C55, C56, C57, C58, C59, C6, C60, C61, C62, C63, C64, C65, C66, C67, C68, C69, C7, C70, C71, C72, C73, C74, C75, C76, C77, C78, C79, C8, C80, C81, C82, C83, C84, C85, C86, C87, C88, C89, C9, C90, C91, C92, C93, C94, C95, C96, C97, C98, C99: 100nF 10V X5R 0402, symbol Device:C
- added R1, R10, R11, R12, R13, R14, R15, R16, R17, R18, R19, R2, R20, R21, R22, R23, R24, R25, R26, R27, R28, R29, R3, R30, R31, R32, R33, R34, R35, R36, R37, R38, R39, R4, R40, R41, R42, R43, R44, R45, R46, R47, R48, R49, R5, R50, R51, R52, R53, R54, R55, R56, R57, R58, R59, R6, R60, R61, R7, R8, R9: 10k 0402, symbol Device:R
- added U1, U10, U11, U12, U13, U14, U15, U16, U17, U18, U19, U2, U20, U21, U22, U23, U24, U25, U26, U27, U28, U29, U3, U30, U31, U32, U33, U34, U35, U36, U37, U38, U39, U4, U40, U41, U42, U43, U44, U45, U46, U47, U48, U49, U5, U50, U51, U52, U53, U54, U55, U56, U57, U58, U59, U6, U60, U61, U7, U8, U9: DRV5055A2QDBZR, symbol PULSAR:DRV5055A2
Connections:
- new net: R13.1, U13.2 (OUT)
- new net: R36.1, U36.2 (OUT)
- new net: R34.1, U34.2 (OUT)
- new net: R20.1, U20.2 (OUT)
- new net: R57.1, U57.2 (OUT)
- new net: R1.1, U1.2 (OUT)
- new net: R49.1, U49.2 (OUT)
- new net: R17.1, U17.2 (OUT)
- new net: R39.1, U39.2 (OUT)
- new net: R27.1, U27.2 (OUT)
- new net: R56.1, U56.2 (OUT)
- new net: R48.1, U48.2 (OUT)
- new net: R10.1, U10.2 (OUT)
- new net: R54.1, U54.2 (OUT)
- new net: R42.1, U42.2 (OUT)
- new net: R47.1, U47.2 (OUT)
- new net: R15.1, U15.2 (OUT)
- new net: R14.1, U14.2 (OUT)
- new net: R58.1, U58.2 (OUT)
- new net: R44.1, U44.2 (OUT)
- new net: R43.1, U43.2 (OUT)
- new net: R55.1, U55.2 (OUT)
- new net: R28.1, U28.2 (OUT)
- new net: R5.1, U5.2 (OUT)
- new net: R52.1, U52.2 (OUT)
- new net: R37.1, U37.2 (OUT)
- new net: R24.1, U24.2 (OUT)
- new net: R46.1, U46.2 (OUT)
- new net: R26.1, U26.2 (OUT)
- new net: R45.1, U45.2 (OUT)
- new net: R29.1, U29.2 (OUT)
- new net: R50.1, U50.2 (OUT)
- new net: R12.1, U12.2 (OUT)
- new net: R32.1, U32.2 (OUT)
- new net: R22.1, U22.2 (OUT)
- new net: R38.1, U38.2 (OUT)
- new net: R4.1, U4.2 (OUT)
- new net: R41.1, U41.2 (OUT)
- new net: R30.1, U30.2 (OUT)
- new net: R33.1, U33.2 (OUT)
- new net: R6.1, U6.2 (OUT)
- new net: R25.1, U25.2 (OUT)
- new net: R11.1, U11.2 (OUT)
- new net: R61.1, U61.2 (OUT)
- new net: R8.1, U8.2 (OUT)
- new net: R40.1, U40.2 (OUT)
- new net: R18.1, U18.2 (OUT)
- new net: R3.1, U3.2 (OUT)
- new net: R35.1, U35.2 (OUT)
- new net: R60.1, U60.2 (OUT)
- new net: R59.1, U59.2 (OUT)
- new net: R16.1, U16.2 (OUT)
- new net: R51.1, U51.2 (OUT)
- new net: R9.1, U9.2 (OUT)
- new net: R19.1, U19.2 (OUT)
- new net: R7.1, U7.2 (OUT)
- new net: R23.1, U23.2 (OUT)
- new net: R53.1, U53.2 (OUT)
- new net: R21.1, U21.2 (OUT)
- new net: R31.1, U31.2 (OUT)
- new net: R2.1, U2.2 (OUT)
- new net +3.3V: U1.1 (VCC), U10.1 (VCC), U11.1 (VCC), U12.1 (VCC), U13.1 (VCC), U14.1 (VCC), U15.1 (VCC), U16.1 (VCC), U17.1 (VCC), U18.1 (VCC), U19.1 (VCC), U2.1 (VCC), U20.1 (VCC), U21.1 (VCC), U22.1 (VCC), U23.1 (VCC), U24.1 (VCC), U25.1 (VCC), U26.1 (VCC), U27.1 (VCC), U28.1 (VCC), U29.1 (VCC), U3.1 (VCC), U30.1 (VCC), U31.1 (VCC), U32.1 (VCC), U33.1 (VCC), U34.1 (VCC), U35.1 (VCC), U36.1 (VCC), U37.1 (VCC), U38.1 (VCC), U39.1 (VCC), U4.1 (VCC), U40.1 (VCC), U41.1 (VCC), U42.1 (VCC), U43.1 (VCC), U44.1 (VCC), U45.1 (VCC), U46.1 (VCC), U47.1 (VCC), U48.1 (VCC), U49.1 (VCC), U5.1 (VCC), U50.1 (VCC), U51.1 (VCC), U52.1 (VCC), U53.1 (VCC), U54.1 (VCC), U55.1 (VCC), U56.1 (VCC), U57.1 (VCC), U58.1 (VCC), U59.1 (VCC), U6.1 (VCC), U60.1 (VCC), U61.1 (VCC), U7.1 (VCC), U8.1 (VCC), U9.1 (VCC)
- new net GND: U1.3 (GND), U10.3 (GND), U11.3 (GND), U12.3 (GND), U13.3 (GND), U14.3 (GND), U15.3 (GND), U16.3 (GND), U17.3 (GND), U18.3 (GND), U19.3 (GND), U2.3 (GND), U20.3 (GND), U21.3 (GND), U22.3 (GND), U23.3 (GND), U24.3 (GND), U25.3 (GND), U26.3 (GND), U27.3 (GND), U28.3 (GND), U29.3 (GND), U3.3 (GND), U30.3 (GND), U31.3 (GND), U32.3 (GND), U33.3 (GND), U34.3 (GND), U35.3 (GND), U36.3 (GND), U37.3 (GND), U38.3 (GND), U39.3 (GND), U4.3 (GND), U40.3 (GND), U41.3 (GND), U42.3 (GND), U43.3 (GND), U44.3 (GND), U45.3 (GND), U46.3 (GND), U47.3 (GND), U48.3 (GND), U49.3 (GND), U5.3 (GND), U50.3 (GND), U51.3 (GND), U52.3 (GND), U53.3 (GND), U54.3 (GND), U55.3 (GND), U56.3 (GND), U57.3 (GND), U58.3 (GND), U59.3 (GND), U6.3 (GND), U60.3 (GND), U61.3 (GND), U7.3 (GND), U8.3 (GND), U9.3 (GND)
- new net HALL0: C2.1, R1.2
- new net HALL1: C4.1, R2.2
- new net HALL10: C22.1, R11.2
- new net HALL11: C24.1, R12.2
- new net HALL12: C26.1, R13.2
- new net HALL13: C28.1, R14.2
- new net HALL14: C30.1, R15.2
- new net HALL15: C32.1, R16.2
- new net HALL16: C34.1, R17.2
- new net HALL17: C36.1, R18.2
- new net HALL18: C38.1, R19.2
- new net HALL19: C40.1, R20.2
- new net HALL2: C6.1, R3.2
- new net HALL20: C42.1, R21.2
- new net HALL21: C44.1, R22.2
- new net HALL22: C46.1, R23.2
- new net HALL23: C48.1, R24.2
- new net HALL24: C50.1, R25.2
- new net HALL25: C52.1, R26.2
- new net HALL26: C54.1, R27.2
- new net HALL27: C56.1, R28.2
- new net HALL28: C58.1, R29.2
- new net HALL29: C60.1, R30.2
- new net HALL3: C8.1, R4.2
- new net HALL30: C62.1, R31.2
- new net HALL31: C64.1, R32.2
- new net HALL32: C66.1, R33.2
- new net HALL33: C68.1, R34.2
- new net HALL34: C70.1, R35.2
- new net HALL35: C72.1, R36.2
- new net HALL36: C74.1, R37.2
- new net HALL37: C76.1, R38.2
- new net HALL38: C78.1, R39.2
- new net HALL39: C80.1, R40.2
- new net HALL4: C10.1, R5.2
- new net HALL40: C82.1, R41.2
- new net HALL41: C84.1, R42.2
- new net HALL42: C86.1, R43.2
- new net HALL43: C88.1, R44.2
- new net HALL44: C90.1, R45.2
- new net HALL45: C92.1, R46.2
- new net HALL46: C94.1, R47.2
- new net HALL47: C96.1, R48.2
- new net HALL48: C98.1, R49.2
- new net HALL49: C100.1, R50.2
- new net HALL5: C12.1, R6.2
- new net HALL50: C102.1, R51.2
- new net HALL51: C104.1, R52.2
- new net HALL52: C106.1, R53.2
- new net HALL53: C108.1, R54.2
- new net HALL54: C110.1, R55.2
- new net HALL55: C112.1, R56.2
- new net HALL56: C114.1, R57.2
- new net HALL57: C116.1, R58.2
- new net HALL58: C118.1, R59.2
- new net HALL59: C120.1, R60.2
- new net HALL6: C14.1, R7.2
- new net HALL60: C122.1, R61.2
- new net HALL7: C16.1, R8.2
- new net HALL8: C18.1, R9.2
- new net HALL9: C20.1, R10.2
Other:
- note added: "Each sensor: 10kΩ series + 100nF shunt RC filter on output"
- note added: "Hall Sensors — 61× DRV5055A2QDBZR (C266131)"
