File: pcb/pulsar /usb.kicad_sch (KiCad schematic)
At the start: 0 parts

Commit message: feat: added the pcb of the pulsar
Parts:
- added C1, C2: 100nF 10V X5R, symbol Device:C
- added J1: USB_C_Receptacle, symbol PULSAR:USB_C_Receptacle
- added R1, R2: 5.1k 0402, symbol Device:R
- added U1: PRTR5V0U2X, symbol PULSAR:PRTR5V0U2X
Connections:
- new net +5V: J1.A4 (VBUS), J1.A9 (VBUS), J1.B4 (VBUS), J1.B9 (VBUS), U1.4 (VBUS)
- new net GND: J1.GND1 (GND), J1.GND2 (GND), J1.SH2 (SHIELD), R1.1, R1.2, R2.2, U1.1 (GND)
- new net USB_DP_RAW: J1.B7 (D~{+})
- no-connect marks 0 -> 2
Other:
- note added: "CC1/CC2 5.1k pull-down -> UFP mode (host detection)"
- note added: "USB-C Receptacle (C165948) + ESD (C12333)"
