File: pcb/pulsar/adc.kicad_sch (KiCad schematic)
At the start: 42 parts, among them U1 REF5025AIDR, U10 ADG1606BRUZ-REEL7, U11 AD7689BCPZRL7, U12 AD7689BCPZRL7, U13 AD7689BCPZRL7, U14 AD7689BCPZRL7, U15 AD7689BCPZRL7, U16 AD7689BCPZRL7, U17 AD7689BCPZRL7, U18 AD7689BCPZRL7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

Commit message: feat: let everything to route
Signed-off-by: Axel Ibarrondo <135344010+Axel84727@users.noreply.github.com>
Parts:
- renumbered C20 to C_ADC0b, C21 to C_ADC0c, C28 to C_ADC1b, C29 to C_ADC1c, C22 to C_ADC2b, C23 to C_ADC2c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
