File: pcb/pulsar/fido2.kicad_sch (KiCad schematic)
At the start: 16 parts, among them J1 FPC_10P_0.5mm, U1 ISO1540DR, U2 STM32L052K8T6, U3 ATECC608B-MAHDA-S

Commit message: feat: let everything to route
Signed-off-by: Axel Ibarrondo <135344010+Axel84727@users.noreply.github.com>
Parts:
- renumbered C6 to C_ATE1, C1 to C_ISO1, C2 to C_ISO2, C3 to C_STM1, C4 to C_STM2, C5 to C_STM3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
