File: pcb/pulsar/fpga_b2.kicad_sch (KiCad schematic)
At the start: 85 parts

Commit message: feat: let everything to route
Signed-off-by: Axel Ibarrondo <135344010+Axel84727@users.noreply.github.com>
Parts:
- renumbered C1 to C200, C9 to C201, C17 to C202, C25 to C203, C33 to C204, C41 to C205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
