File: pcb/pulsar/fpga_c3.kicad_sch (KiCad schematic)
At the start: 12 parts, among them U8 W25Q128JVSIQ, U9 IS61WV102416BLL, Y1 50MHz, Y2 48MHz

Commit message: feat: let everything to route
Signed-off-by: Axel Ibarrondo <135344010+Axel84727@users.noreply.github.com>
Parts:
- renumbered C1 to C_FLASH1, C2 to C_OSC1A, C4 to C_OSC1B, C3 to C_OSC2A, C5 to C_OSC2B, C6 to C_SRAM1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
