File: pcb/pulsar/hall.kicad_sch (KiCad schematic)
At the start: 244 parts, among them U1 DRV5055A2QDBZR, U10 DRV5055A2QDBZR, U11 DRV5055A2QDBZR, U12 DRV5055A2QDBZR, U13 DRV5055A2QDBZR, U14 DRV5055A2QDBZR, U15 DRV5055A2QDBZR, U16 DRV5055A2QDBZR, U17 DRV5055A2QDBZR, U18 DRV5055A2QDBZR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

Commit message: feat: let everything to route
Signed-off-by: Axel Ibarrondo <135344010+Axel84727@users.noreply.github.com>
Parts:
- renumbered C1 to CB_H00, C17 to CB_H01, C33 to CB_H02, C49 to CB_H03, C65 to CB_H04, C81 to CB_H05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
