File: pcb/pulsar/power.kicad_sch (KiCad schematic)
At the start: 25 parts, among them U1 TPS62130, U2 TPS62130, U3 TPS62133, U4 LP2985-1.0, U5 LP2985AIM5-1.2, U6 TLV70225

Commit message: feat: let everything to route
Signed-off-by: Axel Ibarrondo <135344010+Axel84727@users.noreply.github.com>
Parts:
- renumbered C6 to C4, C7 to C_1V0Ma, C4 to C_1V0Mb, C5 to C_1V0Mc, C8 to C_1V2Ma, C9 to C_1V2Mb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
