File: pcb/pulsar/pulsar .kicad_pcb (KiCad board)
At the start: 16 copper layers, 292 x 102 mm, 414 parts, among them J1 GX-C-065 USB-C, J2 FPC-10p 0.5mm, U1 XC7A200T-2FBG484I, U10 PRTR5V0U2X, U3 W25Q128JVSIQ, U9 IS61WV102416BLL, Y1 50MHz_XTAL, Y2 48MHz_XTAL

Commit message: Feat/config layers (#26)
* Configurar DRC, layers y tamaños de pista

* Update pulsar .kicad_prl numeric entries

Adjust several numeric values in pcb/pulsar/pulsar .kicad_prl (updated entries around the listed numeric array). Also remove the stale temporary KiCad lock file pcb/pulsar/~pulsar .kicad_pcb.lck.

* feat: let everything to route

Signed-off-by: Axel Ibarrondo <135344010+Axel84727@users.noreply.github.com>

---------

Signed-off-by: Axel Ibarrondo <135344010+Axel84727@users.noreply.github.com>
Co-authored-by: Axel Ibarrondo <135344010+Axel84727@users.noreply.github.com>
Parts:
- U1: footprint XC7A200T.pretty:FB484/FGB484/FGB484Artix-7_AMD -> XC7A200T:XC7A200T_FBG484
Connections:
- U1 pad A11: (no net) -> GND
- U1 pad A12: (no net) -> GND
- U1 pad A17: (no net) -> +3V3
- U1 pad A2: (no net) -> GND
- U1 pad A22: (no net) -> GND
- U1 pad A3: (no net) -> GND
- U1 pad A5: (no net) -> GND
- U1 pad A7: (no net) -> GND
- U1 pad A9: (no net) -> GND
- U1 pad AA12: (no net) -> GND
- U1 pad AA17: (no net) -> +3V3
- U1 pad AA2: (no net) -> GND
- U1 pad AA22: (no net) -> GND
- U1 pad AA7: (no net) -> +3V3
- U1 pad AB14: (no net) -> +3V3
- U1 pad AB19: (no net) -> GND
- U1 pad AB4: (no net) -> +3V3
- U1 pad AB9: (no net) -> GND
- U1 pad B11: (no net) -> +1V2_MGT
- U1 pad B12: (no net) -> GND
- U1 pad B14: (no net) -> +3V3
- U1 pad B19: (no net) -> GND
- U1 pad B3: (no net) -> GND
- U1 pad B5: (no net) -> +1V2_MGT
- U1 pad B7: (no net) -> +1V2_MGT
- U1 pad B9: (no net) -> +1V2_MGT
- U1 pad C1: (no net) -> +3V3
- U1 pad C10: (no net) -> GND
- U1 pad C12: (no net) -> GND
- U1 pad C16: (no net) -> GND
- U1 pad C21: (no net) -> +3V3
- U1 pad C3: (no net) -> GND
- U1 pad C4: (no net) -> +1V2_MGT
- U1 pad C6: (no net) -> GND
- U1 pad C8: (no net) -> +1V2_MGT
- U1 pad D10: (no net) -> +1V0_MGT
- U1 pad D12: (no net) -> GND
- U1 pad D13: (no net) -> GND
- U1 pad D18: (no net) -> +3V3
- U1 pad D3: (no net) -> GND
- U1 pad D4: (no net) -> GND
- U1 pad D6: (no net) -> +1V0_MGT
- U1 pad D8: (no net) -> GND
- U1 pad E11: (no net) -> GND
- U1 pad E12: (no net) -> +3V3
- U1 pad E15: (no net) -> +3V3
- U1 pad E20: (no net) -> GND
- U1 pad E4: (no net) -> GND
- U1 pad E5: (no net) -> GND
- U1 pad E7: (no net) -> GND
- U1 pad E8: (no net) -> +1V0_MGT
- U1 pad E9: (no net) -> GND
- U1 pad F11: (no net) -> GND
- U1 pad F12: (no net) -> +1V8
- U1 pad F17: (no net) -> GND
- U1 pad F2: (no net) -> +3V3
- U1 pad F22: (no net) -> +3V3
- U1 pad F5: (no net) -> GND
- U1 pad F7: (no net) -> +1V0_MGT
- U1 pad F9: (no net) -> +1V0_MGT
- U1 pad G10: (no net) -> GND
- U1 pad G12: (no net) -> GND
- U1 pad G14: (no net) -> GND
- U1 pad G19: (no net) -> +3V3
- U1 pad G5: (no net) -> GND
- U1 pad G6: (no net) -> GND
- U1 pad G7: (no net) -> GND
- U1 pad G8: (no net) -> GND
- U1 pad G9: (no net) -> GND
- U1 pad H1: (no net) -> GND
- U1 pad H10: (no net) -> +1V0
- U1 pad H11: (no net) -> GND
- U1 pad H12: (no net) -> +1V8
- U1 pad H16: (no net) -> +3V3
- U1 pad H21: (no net) -> GND
- U1 pad H6: (no net) -> +3V3
- U1 pad H7: (no net) -> GND
- U1 pad H8: (no net) -> +1V0
- U1 pad H9: (no net) -> GND
- U1 pad J10: (no net) -> GND
- U1 pad J11: (no net) -> +1V0
- U1 pad J12: (no net) -> GND
- U1 pad J13: (no net) -> +3V3
- U1 pad J18: (no net) -> GND
- U1 pad J3: (no net) -> +3V3
- U1 pad J7: (no net) -> +1V0
- U1 pad J8: (no net) -> GND
- U1 pad J9: (no net) -> +1V0
- U1 pad K10: (no net) -> +1V8
- U1 pad K11: (no net) -> GND
- U1 pad K12: (no net) -> +1V8
- U1 pad K15: (no net) -> GND
- U1 pad K20: (no net) -> +3V3
- U1 pad K5: (no net) -> GND
- U1 pad K7: (no net) -> GND
- U1 pad K8: (no net) -> +1V0
- U1 pad K9: (no net) -> GND
- U1 pad L11: (no net) -> +1V0
- U1 pad L17: (no net) -> +3V3
- U1 pad L2: (no net) -> GND
- U1 pad L22: (no net) -> GND
- U1 pad L7: (no net) -> +1V0
- U1 pad L8: (no net) -> GND
- U1 pad L9: (no net) -> GND
- U1 pad M11: (no net) -> GND
- U1 pad M12: (no net) -> +1V8
- U1 pad M14: (no net) -> +3V3
- U1 pad M19: (no net) -> GND
- U1 pad M4: (no net) -> +3V3
- U1 pad M7: (no net) -> GND
- U1 pad M8: (no net) -> +1V0
- U1 pad N1: (no net) -> +3V3
- U1 pad N11: (no net) -> +1V0
- U1 pad N16: (no net) -> GND
- U1 pad N21: (no net) -> +3V3
- U1 pad N6: (no net) -> GND
- U1 pad N7: (no net) -> +1V0
- U1 pad N8: (no net) -> GND
- U1 pad P10: (no net) -> +1V0
- U1 pad P11: (no net) -> GND
- U1 pad P12: (no net) -> +1V8
- U1 pad P13: (no net) -> GND
- U1 pad P18: (no net) -> +3V3
- U1 pad P3: (no net) -> GND
- U1 pad P7: (no net) -> GND
- U1 pad P8: (no net) -> +1V0
- U1 pad P9: (no net) -> GND
- U1 pad R10: (no net) -> GND
- U1 pad R11: (no net) -> +1V8
- U1 pad R12: (no net) -> GND
- U1 pad R15: (no net) -> +3V3
- U1 pad R20: (no net) -> GND
- U1 pad R5: (no net) -> +3V3
- U1 pad R7: (no net) -> +1V0
- U1 pad R8: (no net) -> GND
- U1 pad R9: (no net) -> +1V0
- U1 pad T10: (no net) -> +1V0
- U1 pad T11: (no net) -> GND
- U1 pad T12: (no net) -> +1V8
- U1 pad T17: (no net) -> GND
- U1 pad T2: (no net) -> +3V3
- U1 pad T22: (no net) -> +3V3
- U1 pad T7: (no net) -> GND
- U1 pad T8: (no net) -> +1V0
- U1 pad T9: (no net) -> GND
- U1 pad U14: (no net) -> GND
- U1 pad U19: (no net) -> +3V3
- U1 pad U4: (no net) -> GND
- U1 pad V1: (no net) -> GND
- U1 pad V11: (no net) -> GND
- U1 pad V16: (no net) -> +3V3
- U1 pad V21: (no net) -> GND
- U1 pad V6: (no net) -> +3V3
- U1 pad W13: (no net) -> +3V3
- U1 pad W18: (no net) -> GND
- U1 pad W3: (no net) -> +3V3
- U1 pad W8: (no net) -> GND
- U1 pad Y10: (no net) -> +3V3
- U1 pad Y15: (no net) -> GND
- U1 pad Y20: (no net) -> +3V3
- U1 pad Y5: (no net) -> GND
- U9 pad 1: (no net) -> SRAM_A0
- U9 pad 10: (no net) -> SRAM_A9
- U9 pad 11: (no net) -> SRAM_OE_N
- U9 pad 12: (no net) -> SRAM_WE_N
- U9 pad 13: (no net) -> SRAM_CE_N
- U9 pad 14: (no net) -> SRAM_D0
- U9 pad 15: (no net) -> SRAM_D1
- U9 pad 16: (no net) -> SRAM_D2
- U9 pad 17: (no net) -> SRAM_D3
- U9 pad 18: (no net) -> SRAM_D4
- U9 pad 19: (no net) -> SRAM_D5
- U9 pad 2: (no net) -> SRAM_A1
- U9 pad 20: (no net) -> SRAM_D6
- U9 pad 21: (no net) -> SRAM_D7
- U9 pad 22: (no net) -> GND
- U9 pad 23: (no net) -> SRAM_A10
- U9 pad 24: (no net) -> SRAM_A11
- U9 pad 25: (no net) -> SRAM_A12
- U9 pad 26: (no net) -> SRAM_A13
- U9 pad 27: (no net) -> SRAM_A14
- U9 pad 28: (no net) -> SRAM_A15
- U9 pad 29: (no net) -> SRAM_A16
- U9 pad 3: (no net) -> SRAM_A2
- U9 pad 30: (no net) -> SRAM_A17
- U9 pad 31: (no net) -> SRAM_A18
- U9 pad 32: (no net) -> SRAM_A19
- U9 pad 33: (no net) -> SRAM_D8
- U9 pad 34: (no net) -> SRAM_D9
- U9 pad 35: (no net) -> SRAM_D10
- U9 pad 36: (no net) -> SRAM_D11
- U9 pad 37: (no net) -> SRAM_D12
- U9 pad 38: (no net) -> SRAM_D13
- U9 pad 39: (no net) -> SRAM_D14
- U9 pad 4: (no net) -> SRAM_A3
- U9 pad 40: (no net) -> SRAM_D15
- U9 pad 41: (no net) -> SRAM_CE2_N
- U9 pad 42: (no net) -> GND
- U9 pad 43: (no net) -> GND
- U9 pad 44: (no net) -> +3V3
- U9 pad 5: (no net) -> SRAM_A4
- U9 pad 6: (no net) -> SRAM_A5
- U9 pad 7: (no net) -> SRAM_A6
- U9 pad 8: (no net) -> SRAM_A7
- U9 pad 9: (no net) -> SRAM_A8
- U_ADC0 pad 11: (no net) -> GND
- U_ADC0 pad 13: (no net) -> GND
- U_ADC0 pad 14: (no net) -> GND
- U_ADC0 pad 15: (no net) -> GND
- U_ADC0 pad 16: (no net) -> GND
- U_ADC0 pad 17: (no net) -> GND
- U_ADC0 pad 18: (no net) -> GND
- U_ADC0 pad 7: +3V3 -> +2V5_REF
- U_ADC0 pad 8: (no net) -> GND
- U_ADC0 pad 9: (no net) -> MUX0_OUT
- U_ADC1 pad 11: (no net) -> GND
- U_ADC1 pad 13: (no net) -> GND
- U_ADC1 pad 14: (no net) -> GND
- U_ADC1 pad 15: (no net) -> GND
- U_ADC1 pad 16: (no net) -> GND
- U_ADC1 pad 17: (no net) -> GND
- U_ADC1 pad 18: (no net) -> GND
- U_ADC1 pad 7: +3V3 -> +2V5_REF
- U_ADC1 pad 8: (no net) -> GND
- U_ADC1 pad 9: (no net) -> MUX1_OUT
- U_ADC2 pad 11: (no net) -> GND
- U_ADC2 pad 13: (no net) -> GND
- U_ADC2 pad 14: (no net) -> GND
- U_ADC2 pad 15: (no net) -> GND
- U_ADC2 pad 16: (no net) -> GND
- U_ADC2 pad 17: (no net) -> GND
- U_ADC2 pad 18: (no net) -> GND
- U_ADC2 pad 7: +3V3 -> +2V5_REF
- U_ADC2 pad 8: (no net) -> GND
- U_ADC2 pad 9: (no net) -> MUX2_OUT
- U_ADC3 pad 11: (no net) -> GND
- U_ADC3 pad 13: (no net) -> GND
- U_ADC3 pad 14: (no net) -> GND
- U_ADC3 pad 15: (no net) -> GND
- U_ADC3 pad 16: (no net) -> GND
- U_ADC3 pad 17: (no net) -> GND
- U_ADC3 pad 18: (no net) -> GND
- U_ADC3 pad 7: +3V3 -> +2V5_REF
- U_ADC3 pad 8: (no net) -> GND
- U_ADC3 pad 9: (no net) -> MUX3_OUT
- U_ADC4 pad 11: (no net) -> GND
- U_ADC4 pad 13: (no net) -> GND
- U_ADC4 pad 14: (no net) -> GND
- U_ADC4 pad 15: (no net) -> GND
- U_ADC4 pad 16: (no net) -> GND
- U_ADC4 pad 17: (no net) -> GND
- U_ADC4 pad 18: (no net) -> GND
- U_ADC4 pad 7: +3V3 -> +2V5_REF
- U_ADC4 pad 8: (no net) -> GND
- U_ADC4 pad 9: (no net) -> MUX0_OUT
- U_ADC5 pad 11: (no net) -> GND
- U_ADC5 pad 13: (no net) -> GND
- U_ADC5 pad 14: (no net) -> GND
- U_ADC5 pad 15: (no net) -> GND
- U_ADC5 pad 16: (no net) -> GND
- U_ADC5 pad 17: (no net) -> GND
- U_ADC5 pad 18: (no net) -> GND
- U_ADC5 pad 7: +3V3 -> +2V5_REF
- U_ADC5 pad 8: (no net) -> GND
- U_ADC5 pad 9: (no net) -> MUX1_OUT
- U_ADC6 pad 11: (no net) -> GND
- U_ADC6 pad 13: (no net) -> GND
- U_ADC6 pad 14: (no net) -> GND
- U_ADC6 pad 15: (no net) -> GND
- U_ADC6 pad 16: (no net) -> GND
- U_ADC6 pad 17: (no net) -> GND
- U_ADC6 pad 18: (no net) -> GND
- U_ADC6 pad 7: +3V3 -> +2V5_REF
- U_ADC6 pad 8: (no net) -> GND
- U_ADC6 pad 9: (no net) -> MUX2_OUT
- U_ADC7 pad 11: (no net) -> GND
- U_ADC7 pad 13: (no net) -> GND
- U_ADC7 pad 14: (no net) -> GND
- U_ADC7 pad 15: (no net) -> GND
- U_ADC7 pad 16: (no net) -> GND
- U_ADC7 pad 17: (no net) -> GND
- U_ADC7 pad 18: (no net) -> GND
- U_ADC7 pad 7: +3V3 -> +2V5_REF
- U_ADC7 pad 8: (no net) -> GND
- U_ADC7 pad 9: (no net) -> MUX3_OUT
- U_BUF0 pad 1: (no net) -> MUX0_OUT
- U_BUF0 pad 2: (no net) -> GND
- U_BUF0 pad 3: (no net) -> MUX0_D
- U_BUF0 pad 4: GND -> MUX0_OUT
- U_BUF1 pad 1: (no net) -> MUX1_OUT
- U_BUF1 pad 2: (no net) -> GND
- U_BUF1 pad 3: (no net) -> MUX1_D
- U_BUF1 pad 4: GND -> MUX1_OUT
- U_BUF2 pad 1: (no net) -> MUX2_OUT
- U_BUF2 pad 2: (no net) -> GND
- U_BUF2 pad 3: (no net) -> MUX2_D
- U_BUF2 pad 4: GND -> MUX2_OUT
- U_BUF3 pad 1: (no net) -> MUX3_OUT
- U_BUF3 pad 2: (no net) -> GND
- U_BUF3 pad 3: (no net) -> MUX3_D
- U_BUF3 pad 4: GND -> MUX3_OUT
- U_MUX0 pad 1: (no net) -> HALL0
- U_MUX0 pad 10: (no net) -> HALL9
- U_MUX0 pad 11: (no net) -> HALL10
- U_MUX0 pad 12: (no net) -> HALL11
- U_MUX0 pad 13: (no net) -> HALL12
- U_MUX0 pad 14: (no net) -> HALL13
- U_MUX0 pad 15: (no net) -> GND
- U_MUX0 pad 16: (no net) -> HALL14
- U_MUX0 pad 17: (no net) -> HALL15
- U_MUX0 pad 18: (no net) -> MUX_A0
- U_MUX0 pad 19: (no net) -> MUX_A1
- U_MUX0 pad 2: (no net) -> HALL1
- U_MUX0 pad 20: (no net) -> MUX_A2
- U_MUX0 pad 21: (no net) -> MUX_A3
- U_MUX0 pad 22: (no net) -> MUX0_EN
- U_MUX0 pad 23: (no net) -> MUX0_D
- U_MUX0 pad 24: (no net) -> +3V3
- U_MUX0 pad 3: (no net) -> HALL2
- U_MUX0 pad 4: (no net) -> HALL3
- U_MUX0 pad 5: (no net) -> HALL4
- U_MUX0 pad 6: (no net) -> HALL5
- U_MUX0 pad 7: (no net) -> HALL6
- U_MUX0 pad 8: (no net) -> HALL7
- U_MUX0 pad 9: (no net) -> HALL8
- U_MUX1 pad 1: (no net) -> HALL16
- U_MUX1 pad 10: (no net) -> HALL25
- U_MUX1 pad 11: (no net) -> HALL26
- U_MUX1 pad 12: (no net) -> HALL27
- U_MUX1 pad 13: (no net) -> HALL28
- U_MUX1 pad 14: (no net) -> HALL29
- U_MUX1 pad 15: (no net) -> GND
- U_MUX1 pad 16: (no net) -> HALL30
- U_MUX1 pad 17: (no net) -> HALL31
- U_MUX1 pad 18: (no net) -> MUX_A0
- U_MUX1 pad 19: (no net) -> MUX_A1
- U_MUX1 pad 2: (no net) -> HALL17
- U_MUX1 pad 20: (no net) -> MUX_A2
- U_MUX1 pad 21: (no net) -> MUX_A3
- U_MUX1 pad 22: (no net) -> MUX1_EN
- U_MUX1 pad 23: (no net) -> MUX1_D
- U_MUX1 pad 24: (no net) -> +3V3
- U_MUX1 pad 3: (no net) -> HALL18
- U_MUX1 pad 4: (no net) -> HALL19
- U_MUX1 pad 5: (no net) -> HALL20
- U_MUX1 pad 6: (no net) -> HALL21
- U_MUX1 pad 7: (no net) -> HALL22
- U_MUX1 pad 8: (no net) -> HALL23
- U_MUX1 pad 9: (no net) -> HALL24
- U_MUX2 pad 1: (no net) -> HALL32
- U_MUX2 pad 10: (no net) -> HALL41
- U_MUX2 pad 11: (no net) -> HALL42
- U_MUX2 pad 12: (no net) -> HALL43
- U_MUX2 pad 13: (no net) -> HALL44
- U_MUX2 pad 14: (no net) -> HALL45
- U_MUX2 pad 15: (no net) -> GND
- U_MUX2 pad 16: (no net) -> HALL46
- U_MUX2 pad 17: (no net) -> HALL47
- U_MUX2 pad 18: (no net) -> MUX_A0
- U_MUX2 pad 19: (no net) -> MUX_A1
- U_MUX2 pad 2: (no net) -> HALL33
- U_MUX2 pad 20: (no net) -> MUX_A2
- U_MUX2 pad 21: (no net) -> MUX_A3
- U_MUX2 pad 22: (no net) -> MUX2_EN
- U_MUX2 pad 23: (no net) -> MUX2_D
- U_MUX2 pad 24: (no net) -> +3V3
- U_MUX2 pad 3: (no net) -> HALL34
- U_MUX2 pad 4: (no net) -> HALL35
- U_MUX2 pad 5: (no net) -> HALL36
- U_MUX2 pad 6: (no net) -> HALL37
- U_MUX2 pad 7: (no net) -> HALL38
- U_MUX2 pad 8: (no net) -> HALL39
- U_MUX2 pad 9: (no net) -> HALL40
- U_MUX3 pad 1: (no net) -> HALL48
- U_MUX3 pad 10: (no net) -> HALL57
- U_MUX3 pad 11: (no net) -> HALL58
- U_MUX3 pad 12: (no net) -> HALL59
- U_MUX3 pad 13: (no net) -> HALL60
- U_MUX3 pad 15: (no net) -> GND
- U_MUX3 pad 18: (no net) -> MUX_A0
- U_MUX3 pad 19: (no net) -> MUX_A1
- U_MUX3 pad 2: (no net) -> HALL49
- U_MUX3 pad 20: (no net) -> MUX_A2
- U_MUX3 pad 21: (no net) -> MUX_A3
- U_MUX3 pad 22: (no net) -> MUX3_EN
- U_MUX3 pad 23: (no net) -> MUX3_D
- U_MUX3 pad 24: (no net) -> +3V3
- U_MUX3 pad 3: (no net) -> HALL50
- U_MUX3 pad 4: (no net) -> HALL51
- U_MUX3 pad 5: (no net) -> HALL52
- U_MUX3 pad 6: (no net) -> HALL53
- U_MUX3 pad 7: (no net) -> HALL54
- U_MUX3 pad 8: (no net) -> HALL55
- U_MUX3 pad 9: (no net) -> HALL56
- U_REF0 pad 5: +3V3 -> +2V5_REF
- U_REF0 pad 6: (no net) -> +3V3
- U_REF0 pad 8: +3V3 -> +2V5_REF
- U_REF1 pad 5: +3V3 -> +2V5_REF
- U_REF1 pad 6: (no net) -> +3V3
- U_REF1 pad 8: +3V3 -> +2V5_REF
- U_STM pad 1: (no net) -> +3V3
- U_STM pad 16: (no net) -> GND
- U_STM pad 17: (no net) -> GND
- U_STM pad 18: (no net) -> USB_DM_RAW
- U_STM pad 19: (no net) -> USB_DP_RAW
- U_STM pad 20: (no net) -> SWDIO
- U_STM pad 21: (no net) -> SWCLK
- U_STM pad 29: (no net) -> FIDO2_SCL
- U_STM pad 30: (no net) -> FIDO2_SDA
- U_STM pad 31: (no net) -> GND
- U_STM pad 32: (no net) -> +3V3
- U_STM pad 4: (no net) -> NRST_STM
Routing:
- added copper zone on In3.Cu, net +1V0
- added copper zone on In10.Cu, net +1V0_MGT
- added copper zone on In5.Cu, net +1V8
- added copper zone on In12.Cu, net +3V3
- added copper zone on B.Cu, net GND
- added copper zone on F.Cu, net GND
- added copper zone on In1.Cu, net GND
- added copper zone on In14.Cu, net GND
- added copper zone on In7.Cu, net GND
- added copper zone on In8.Cu, net GND
